File: Parkplatz/Parkplatz.kicad_pcb (KiCad board)
At the start: 2 copper layers, 42.2 x 17.5 mm, 6 parts, among them J1 Conn_01x06_Female

Commit message: Modul überarbeitet
Parts:
- added J2: Conn_01x03_Female, Connector_PinSocket_2.54mm:PinSocket_1x03_P2.54mm_Vertical, F.Cu at (160.0, 98.4)
- J1: footprint Connector_PinSocket_2.54mm:PinSocket_1x06_P2.54mm_Vertical -> Connector_PinHeader_2.54mm:PinHeader_1x06_P2.54mm_Vertical
- moved R1 10.0 mm to (152.0, 102.0)
- moved R2 4.95 mm to (151.9, 99.4)
- moved J1 2.71 mm to (147.3, 94.4)
- moved R4 2.67 mm to (151.9, 104.5)
- moved D1 1.17 mm to (181.9, 98.9), turned to 270 degrees
- moved R3 0.64 mm to (151.9, 96.9)
Connections:
- J1 pad 1: Net-(J1-Pad1) -> Net-(D1-Pad2)
- J1 pad 5: Net-(D1-Pad2) -> Net-(J1-Pad5)
- R1 pad 1: Net-(J1-Pad1) -> Net-(J1-Pad4)
- R2 pad 1: Net-(J1-Pad2) -> Net-(J1-Pad3)
- R3 pad 1: Net-(J1-Pad3) -> Net-(J1-Pad2)
- R4 pad 1: Net-(J1-Pad4) -> Net-(J1-Pad5)
Routing:
- net Net-(D1-Pad2): track 50.6 -> 73.8 mm
- net Net-(J1-Pad5): track 0.00 -> 16.5 mm
- net Net-(J1-Pad6): track 14.9 -> 28.8 mm
- net Net-(J1-Pad4): track 16.7 -> 3.18 mm
- net Net-(D1-Pad3): track 29.5 -> 35.5 mm
- net Net-(D1-Pad4): track 30.0 -> 35.4 mm
- net Net-(J1-Pad1): track 3.84 -> 0.00 mm
- net Net-(D1-Pad1): track 30.1 -> 32.0 mm
- net Net-(J1-Pad3): track 3.84 -> 3.12 mm
- net Net-(J1-Pad2): track 3.56 -> 3.05 mm
- added copper zone on B.Cu, net Net-(J1-Pad6)
- removed copper zone on B.Cu, net (none)
Other:
- board size 42.2 x 17.5 mm -> 42.2 x 22.4 mm
- board text added: "Durchmesser von bolzen nochmal messen und im PCB ändern"
- board text added: "M.S"
- board text added: "Parkplatz v.0.4"
- board text removed: "Parkplatz v.0.3"

Commit message: Verbesserung fehlt
Other:
- board text removed: "Durchmesser von bolzen nochmal messen und im PCB ändern"
Changed lines of the file:
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@@
-(kicad_pcb (version 20171130) (host pcbnew "(5.1.5)-2")
+(kicad_pcb (version 20171130) (host pcbnew "(5.1.4)-1")
   (general
     (thickness 1.6)
-    (drawings 16)
+    (drawings 15)
     (tracks 57)
     (zones 0)
@@
     )
   )
-  (gr_text "Durchmesser von bolzen nochmal messen und im PCB ändern" (at 168.402 100.33) (layer B.Cu)
-    (effects (font (size 1.5 1.5) (thickness 0.3)) (justify mirror))
-  )
-  (gr_text M.S (at 177.546 109.728) (layer B.Cu)
+  (gr_circle (center 181.61 107.886) (end 183.96 107.886) (layer B.SilkS) (width 0.15))
+  (gr_circle (center 181.61 92.773) (end 183.96 92.773) (layer B.SilkS) (width 0.15))
+  (gr_text M.S (at 171.831 94.107) (layer B.Cu)
     (effects (font (size 1 1) (thickness 0.25)) (justify mirror))
   )
@@
   (gr_line (start 144.272 111.76) (end 186.436 111.76) (layer Edge.Cuts) (width 0.15))
   (gr_line (start 144.272 106.934) (end 144.272 110.236) (layer Edge.Cuts) (width 0.15))
-  (gr_circle (center 181.61 107.95) (end 183.134 107.95) (layer B.SilkS) (width 0.15))
-  (gr_circle (center 181.61 92.7735) (end 183.134 92.7735) (layer B.SilkS) (width 0.15))
-  (gr_text "Parkplatz v.0.4\n" (at 170.18 107.696) (layer B.Cu)
+  (gr_text "Parkplatz v.0.4\n" (at 170.053 91.694) (layer B.Cu)
     (effects (font (size 1.5 1.5) (thickness 0.3)) (justify mirror))
   )
@@
       )
     )
+  )
+  (zone (net 0) (net_name "") (layer B.Cu) (hatch edge 0.508)
+    (connect_pads (clearance 0.508))
+    (min_thickness 0.254)
+    (keepout (tracks allowed) (vias allowed) (copperpour not_allowed))
+    (fill (arc_segments 32) (thermal_gap 0.508) (thermal_bridge_width 0.508))
+    (polygon
+      (pts
+        (xy 149.479 95.758) (xy 154.305 95.758) (xy 154.305 105.664) (xy 149.479 105.664) (xy 149.352 95.758)
+      )
+    )
