File: MainPL/MainPL.sch (KiCad schematic (older format))
At the start: 39 parts, among them J1 Conn_01x06_Female, J10 Conn_01x06_Female, J11 Conn_01x06_Female, J12 Conn_01x06_Female, J13 Conn_01x06_Female, J14 Conn_01x06_Female, J15 Conn_01x01_Male, J2 USB_B, J3 Conn_01x06_Female, J4 Conn_01x06_Female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

Commit message: Add files via upload
Parts:
- removed SW1: SW_DIP_x02, Button_Switch_THT:SW_TH_Tactile_Omron_B3F-10xx, symbol Switch:SW_DIP_x02
- removed U6, U8, U9: 74LS32, symbol 74xx:74LS32
- removed U?: 74LS573, symbol 74xx:74LS573
- added SW1: SW_Push_Dual, symbol Switch:SW_Push_Dual
- added U6: 74LS373, symbol 74xx:74LS373
- added U8: MC74HC589A, symbol Buffer_74HC589:MC74HC589A
Connections:
- net labels added: CP, LE, OE, Q7, ^CE, ^PL
- net labels removed: INTA_1, INTA_2, INTA_3
- wire segments 283 -> 295
Other:
- note added: "NICHT FERTIG!!\n"
- moved on the sheet: C4, D1, J15, R7, U2

Commit message: Add files via upload
Schaltplan fertig
Parts:
- removed J7: Conn_01x04_Female, Connector_PinHeader_2.54mm:PinHeader_1x04_P2.54mm_Vertical, symbol Connector:Conn_01x04_Female
- removed U10, U3, U7: MCP23017_ML, Package_DFN_QFN:QFN-28-1EP_6x6mm_P0.65mm_EP4.25x4.25mm, symbol Interface_Expansion:MCP23017_ML
- removed U5: Display_16x2_I2C, MainPL_LCD:16x2_LCD_I2C, symbol display_16x2_i2c:Display_16x2_I2C
- added J16: Conn_01x04_Male, Connector_PinHeader_2.54mm:PinHeader_1x04_P2.54mm_Vertical, symbol Connector:Conn_01x04_Male
- added J7: Conn_01x09_Male, Connector_PinHeader_2.54mm:PinHeader_1x09_P2.54mm_Horizontal, symbol Connector:Conn_01x09_Male
- added U3, U5, U7: MCP23017_SP, Package_DIP:DIP-28_W7.62mm_Socket_LongPads, symbol Interface_Expansion:MCP23017_SP
- added U9: 74LVC2G04, Package_DIP:DIP-6_W7.62mm_Socket_LongPads, symbol 74xGxx:74LVC2G04
- R1, R2, R3, R4, R6, R8: footprint (none) -> Resistor_SMD:R_1206_3216Metric_Pad1.42x1.75mm_HandSolder
- SW1: footprint (none) -> Button_Switch_THT:SW_TH_Tactile_Omron_B3F-10xx
- U1, U4: footprint (none) -> Package_DIP:DIP-14_W7.62mm_Socket_LongPads
- U6: footprint (none) -> Package_DIP:DIP-20_W7.62mm_Socket_LongPads
- U8: footprint (none) -> Package_DIP:DIP-16_W7.62mm_Socket_LongPads
Connections:
- net labels added: CLK, CLK_INH, Qh
- net labels removed: CP, Q7, ^CE, ^PL
- wire segments 295 -> 298
Other:
- note added: "5V???\n"
- note added: "Buffer"
- note added: "Delay"
- note removed: "NICHT FERTIG!!\n"
- note removed: "Schauen bei welchen Vcc\n"
- moved on the sheet: U8

Commit message: Add files via upload
Parts:
- removed U4: 74LS32, Package_DIP:DIP-14_W7.62mm_Socket_LongPads, symbol 74xx:74LS32
- added unit 2 of U1
- U2: symbol MCU_Microchip_ATmega:ATmega328P-PU -> MainPL-rescue:ATmega328P-PU-MCU_Microchip_ATmega
Connections:
- net INTArduino: now also U1.6
- net INTB_3: now also U1.4
- net at U1.3: now also U1.5
Changed lines of the file:
@@
 EESchema Schematic File Version 4
-LIBS:MainPL-cache
 EELAYER 30 0
 EELAYER END
@@
 Servo
 $Comp
-L MCU_Microchip_ATmega:ATmega328P-PU U2
+L MainPL-rescue:ATmega328P-PU-MCU_Microchip_ATmega U2
 U 1 1 5DE0CE2B
 P 6950 7775
@@
 Wire Wire Line
 	4150 2975 4425 2975
-$Comp
-L 74xx:74LS32 U4
-U 1 1 5E06A540
-P 5000 6300
-F 0 "U4" V 4954 6488 50  0000 L CNN
-F 1 "74LS32" V 5045 6488 50  0000 L CNN
-F 2 "Package_DIP:DIP-14_W7.62mm_Socket_LongPads" H 5000 6300 50  0001 C CNN
-F 3 "http://www.ti.com/lit/gpn/sn74LS32" H 5000 6300 50  0001 C CNN
-	1    5000 6300
-	0    1    1    0
-$EndComp
 Connection ~ 6575 3900
 Wire Wire Line
@@
 Wire Bus Line
 	6950 5650 6950 6775
-Wire Bus Line
-	1250 2225 1250 5650
-Wire Bus Line
-	6225 3400 6225 5650
-Wire Bus Line
-	3725 2475 3725 5650
-Wire Bus Line
-	3275 5650 3275 7325
-Wire Bus Line
-	1250 5650 3275 5650
-Wire Bus Line
-	9150 4975 9150 5600
-Wire Bus Line
-	12525 4500 12525 6900
-Wire Bus Line
-	7550 6900 10325 6900
-Wire Bus Line
-	3325 7625 3325 9150
-Wire Bus Line
-	8750 3175 12550 3175
-Wire Bus Line
-	8750 3175 8750 4800
-Wire Bus Line
-	6175 2225 9825 2225
-Wire Bus Line
-	6175 2225 6175 3875
-Wire Bus Line
-	3675 1250 3675 3625
-Wire Bus Line
-	3675 1250 7450 1250
 $Comp
 L Interface_Expansion:MCP23017_SP U3
@@
 	1    0    0    -1
 $EndComp
+Wire Bus Line
+	1250 2225 1250 5650
+Wire Bus Line
+	6225 3400 6225 5650
+Wire Bus Line
+	3725 2475 3725 5650
+Wire Bus Line
+	3275 5650 3275 7325
+Wire Bus Line
+	1250 5650 3275 5650
+Wire Bus Line
+	9150 4975 9150 5600
+Wire Bus Line
+	12525 4500 12525 6900
+Wire Bus Line
+	7550 6900 10325 6900
+Wire Bus Line
+	3325 7625 3325 9150
+Wire Bus Line
+	8750 3175 12550 3175
+Wire Bus Line
+	8750 3175 8750 4800
+Wire Bus Line
+	6175 2225 9825 2225
+Wire Bus Line
+	6175 2225 6175 3875
+Wire Bus Line
+	3675 1250 3675 3625
+Wire Bus Line
+	3675 1250 7450 1250
+$Comp
+L 74xx:74LS32 U1
+U 2 1 5E02EBD5
+P 5000 6300
+F 0 "U1" V 4954 6488 50  0000 L CNN
+F 1 "74LS32" V 5045 6488 50  0000 L CNN
+F 2 "Package_DIP:DIP-14_W7.62mm_Socket_LongPads" H 5000 6300 50  0001 C CNN
+F 3 "http://www.ti.com/lit/gpn/sn74LS32" H 5000 6300 50  0001 C CNN
+	2    5000 6300
+	0    1    1    0
+$EndComp
 $EndSCHEMATC

Commit message: Pcb weiter
Parts:
- J15: footprint Connector_PinHeader_2.54mm:PinHeader_1x01_P2.54mm_Vertical -> Connector_PinHeader_2.54mm:PinHeader_1x01_P2.54mm_Horizontal
- J16: footprint Connector_PinHeader_2.54mm:PinHeader_1x04_P2.54mm_Vertical -> Connector_PinHeader_2.54mm:PinHeader_1x04_P2.54mm_Horizontal
Connections:
- net B1: now also U3.3 (GPB2); no longer U3.25 (GPA4)
- net B10: now also U7.7 (GPB6); no longer U7.26 (GPA5)
- net B11: now also U7.22 (GPA1); no longer U7.27 (GPA6)
- net B12: now also U7.26 (GPA5); no longer U7.28 (GPA7)
- net B2: now also U3.7 (GPB6); no longer U3.26 (GPA5)
- net B3: now also U3.22 (GPA1); no longer U3.27 (GPA6)
- net B4: now also U3.26 (GPA5); no longer U3.28 (GPA7)
- net B5: now also U5.3 (GPB2); no longer U5.25 (GPA4)
- net B6: now also U5.7 (GPB6); no longer U5.26 (GPA5)
- net B7: now also U5.22 (GPA1); no longer U5.27 (GPA6)
- net B8: now also U5.26 (GPA5); no longer U5.28 (GPA7)
- net B9: now also U7.3 (GPB2); no longer U7.25 (GPA4)
- net DATA1: now also U3.4 (GPB3); no longer U3.1 (GPB0)
- net DATA10: now also U7.8 (GPB7); no longer U7.2 (GPB1)
- net DATA11: now also U7.21 (GPA0); no longer U7.3 (GPB2)
- net DATA12: now also U7.25 (GPA4); no longer U7.4 (GPB3)
- net DATA2: now also U3.8 (GPB7); no longer U3.2 (GPB1)
- net DATA3: now also U3.21 (GPA0); no longer U3.3 (GPB2)
- net DATA4: now also U3.25 (GPA4); no longer U3.4 (GPB3)
- net DATA5: now also U5.4 (GPB3); no longer U5.1 (GPB0)
- net DATA6: now also U5.8 (GPB7); no longer U5.2 (GPB1)
- net DATA7: now also U5.21 (GPA0); no longer U5.3 (GPB2)
- net DATA8: now also U5.25 (GPA4); no longer U5.4 (GPB3)
- net DATA9: now also U7.4 (GPB3); no longer U7.1 (GPB0)
- net G1: now also U3.2 (GPB1); no longer U3.21 (GPA0)
- net G10: now also U7.6 (GPB5); no longer U7.22 (GPA1)
- net G12: now also U7.27 (GPA6); no longer U7.24 (GPA3)
- net G2: now also U3.6 (GPB5); no longer U3.22 (GPA1)
- net G4: now also U3.27 (GPA6); no longer U3.24 (GPA3)
- net G5: now also U5.2 (GPB1); no longer U5.21 (GPA0)
- net G6: now also U5.6 (GPB5); no longer U5.22 (GPA1)
- net G8: now also U5.27 (GPA6); no longer U5.24 (GPA3)
- net G9: now also U7.2 (GPB1); no longer U7.21 (GPA0)
- net R1: now also U3.1 (GPB0); no longer U3.5 (GPB4)
- net R10: now also U7.5 (GPB4); no longer U7.6 (GPB5)
- net R11: now also U7.24 (GPA3); no longer U7.7 (GPB6)
- net R12: now also U7.28 (GPA7); no longer U7.8 (GPB7)
- net R2: now also U3.5 (GPB4); no longer U3.6 (GPB5)
- net R3: now also U3.24 (GPA3); no longer U3.7 (GPB6)
- net R4: now also U3.28 (GPA7); no longer U3.8 (GPB7)
- net R5: now also U5.1 (GPB0); no longer U5.5 (GPB4)
- net R6: now also U5.5 (GPB4); no longer U5.6 (GPB5)
- net R7: now also U5.24 (GPA3); no longer U5.7 (GPB6)
- net R8: now also U5.28 (GPA7); no longer U5.8 (GPB7)
- net R9: now also U7.1 (GPB0); no longer U7.5 (GPB4)
Other:
- note added: "LCD-Display"
- note removed: "5V???\n"
Changed lines of the file:
@@
 Text Label 4850 1075 1    50   ~ 0
 G2
-Text Label 3325 3525 0    50   ~ 0
-B2
 Text Label 5050 1075 1    50   ~ 0
 DATA2
@@
 Wire Wire Line
 	3300 3725 3575 3725
-Text Label 3325 2125 0    50   ~ 0
-DATA1
-Text Label 3325 2225 0    50   ~ 0
-DATA2
-Text Label 3325 2325 0    50   ~ 0
-DATA3
-Text Label 3325 2425 0    50   ~ 0
-DATA4
-Text Label 3425 2525 2    50   ~ 0
-R1
-Text Label 3325 2625 0    50   ~ 0
-R2
-Text Label 3325 2725 0    50   ~ 0
-R3
-Text Label 3325 2825 0    50   ~ 0
-R4
-Text Label 3325 3025 0    50   ~ 0
-G1
-Text Label 3325 3125 0    50   ~ 0
-G2
-Text Label 3325 3225 0    50   ~ 0
-G3
-Text Label 3325 3325 0    50   ~ 0
-G4
-Text Label 3325 3425 0    50   ~ 0
-B1
-Text Label 3325 3625 0    50   ~ 0
-B3
-Text Label 3325 3725 0    50   ~ 0
-B4
 $Comp
 L power:+5V #PWR019
@@
 Wire Wire Line
 	9725 1825 9725 2125
-Text Label 5850 2375 0    50   ~ 0
-DATA5
-Text Label 5850 2475 0    50   ~ 0
-DATA6
-Text Label 5850 2575 0    50   ~ 0
-DATA7
-Text Label 5850 2675 0    50   ~ 0
-DATA8
-Text Label 5850 2775 0    50   ~ 0
-R5
-Text Label 5850 2875 0    50   ~ 0
-R6
-Text Label 5850 2975 0    50   ~ 0
-R7
-Text Label 5850 3075 0    50   ~ 0
-R8
-Text Label 5850 3275 0    50   ~ 0
-G5
-Text Label 5850 3375 0    50   ~ 0
-G6
-Text Label 5850 3475 0    50   ~ 0
-G7
-Text Label 5850 3575 0    50   ~ 0
-G8
-Text Label 5850 3675 0    50   ~ 0
-B5
-Text Label 5850 3775 0    50   ~ 0
-B6
-Text Label 5850 3875 0    50   ~ 0
-B7
-Text Label 5850 3975 0    50   ~ 0
-B8
 $Comp
 L Connector:Conn_01x06_Female J10
@@
 Text Label 12450 3050 1    50   ~ 0
 DATA12
-Text Label 8350 3300 0    50   ~ 0
-DATA9
-Text Label 8350 3400 0    50   ~ 0
-DATA10
-Text Label 8350 3500 0    50   ~ 0
-DATA11
-Text Label 8350 3600 0    50   ~ 0
-DATA12
-Text Label 8350 3700 0    50   ~ 0
-R9
-Text Label 8350 3800 0    50   ~ 0
-R10
-Text Label 8350 3900 0    50   ~ 0
-R11
-Text Label 8350 4000 0    50   ~ 0
-R12
-Text Label 8350 4200 0    50   ~ 0
-G9
-Text Label 8350 4300 0    50   ~ 0
-G10
-Text Label 8350 4400 0    50   ~ 0
-G11
-Text Label 8350 4500 0    50   ~ 0
-G12
-Text Label 8350 4600 0    50   ~ 0
-B9
-Text Label 8350 4700 0    50   ~ 0
-B10
-Text Label 8350 4800 0    50   ~ 0
-B11
-Text Label 8350 4900 0    50   ~ 0
-B12
 Text Label 2850 7325 0    50   ~ 0
 SCL
@@
 F 0 "J15" H 9522 6957 50  0000 R CNN
 F 1 "Conn_01x01_Male" H 9522 7048 50  0000 R CNN
-F 2 "Connector_PinHeader_2.54mm:PinHeader_1x01_P2.54mm_Vertical" H 9550 7025 50  0001 C CNN
+F 2 "Connector_PinHeader_2.54mm:PinHeader_1x01_P2.54mm_Horizontal" H 9550 7025 50  0001 C CNN
 F 3 "~" H 9550 7025 50  0001 C CNN
 	1    9550 7025
@@
 Text Label 7850 7150 1    39   ~ 0
 CLK_INH
-Text Notes 12175 6100 0    50   ~ 0
-5V???\n
 Wire Notes Line
 	11525 5475 12475 5475
@@
 F 0 "J16" V 1504 5937 50  0000 R CNN
 F 1 "Conn_01x04_Male" V 1413 5937 50  0000 R CNN
-F 2 "Connector_PinHeader_2.54mm:PinHeader_1x04_P2.54mm_Vertical" H 1350 6225 50  0001 C CNN
+F 2 "Connector_PinHeader_2.54mm:PinHeader_1x04_P2.54mm_Horizontal" H 1350 6225 50  0001 C CNN
 F 3 "~" H 1350 6225 50  0001 C CNN
 	1    1350 6225
@@
 	1    0    0    -1
 $EndComp
-Wire Bus Line
-	1250 2225 1250 5650
-Wire Bus Line
-	6225 3400 6225 5650
-Wire Bus Line
-	3725 2475 3725 5650
-Wire Bus Line
-	3275 5650 3275 7325
-Wire Bus Line
-	1250 5650 3275 5650
-Wire Bus Line
-	9150 4975 9150 5600
-Wire Bus Line
-	12525 4500 12525 6900
-Wire Bus Line
-	7550 6900 10325 6900
-Wire Bus Line
-	3325 7625 3325 9150
-Wire Bus Line
-	8750 3175 12550 3175
-Wire Bus Line
-	8750 3175 8750 4800
-Wire Bus Line
-	6175 2225 9825 2225
-Wire Bus Line
-	6175 2225 6175 3875
-Wire Bus Line
-	3675 1250 3675 3625
-Wire Bus Line
-	3675 1250 7450 1250
 $Comp
 L 74xx:74LS32 U1
@@
 	0    1    1    0
 $EndComp
+Text Label 3425 2125 2    50   ~ 0
+R1
+Text Label 3325 2225 0    50   ~ 0
+G1
+Text Label 3325 2525 0    50   ~ 0
+R2
+Text Label 3325 2625 0    50   ~ 0
+G2
+Text Label 3325 2825 0    50   ~ 0
+DATA2
+Text Label 3325 2725 0    50   ~ 0
+B2
+Text Label 3325 2325 0    50   ~ 0
+B1
+Text Label 3325 2425 0    50   ~ 0
+DATA1
+Text Label 3325 3025 0    50   ~ 0
+DATA3
+Text Label 3325 3125 0    50   ~ 0
+B3
+Text Label 3325 3225 0    50   ~ 0
+G3
+Text Label 3325 3325 0    50   ~ 0
+R3
+Text Label 3325 3425 0    50   ~ 0
+DATA4
+Text Label 3325 3525 0    50   ~ 0
+B4
+Text Label 3325 3625 0    50   ~ 0
+G4
+Text Label 3325 3725 0    50   ~ 0
+R4
+Text Label 5850 2375 0    50   ~ 0
+R5
+Text Label 5850 2475 0    50   ~ 0
+G5
+Text Label 5850 2575 0    50   ~ 0
+B5
+Text Label 5850 2675 0    50   ~ 0
+DATA5
+Text Label 5850 2775 0    50   ~ 0
+R6
+Text Label 5850 2875 0    50   ~ 0
+G6
+Text Label 5850 2975 0    50   ~ 0
+B6
+Text Label 5850 3075 0    50   ~ 0
+DATA6
+Text Label 8375 3300 0    50   ~ 0
+R9
+Text Label 8375 3400 0    50   ~ 0
+G9
+Text Label 5850 3275 0    50   ~ 0
+DATA7
+Text Label 5850 3375 0    50   ~ 0
+B7
+Text Label 5850 3475 0    50   ~ 0
+G7
+Text Label 5850 3575 0    50   ~ 0
+R7
+Text Label 5850 3675 0    50   ~ 0
+DATA8
+Text Label 5850 3775 0    50   ~ 0
+B8
+Text Label 5850 3875 0    50   ~ 0
+G8
+Text Label 5850 3975 0    50   ~ 0
+R8
+Text Label 8375 3500 0    50   ~ 0
+B9
+Text Label 8375 3600 0    50   ~ 0
+DATA9
+Text Label 8375 3700 0    50   ~ 0
+R10
+Text Label 8375 3800 0    50   ~ 0
+G10
+Text Label 8375 3900 0    50   ~ 0
+B10
+Text Label 8375 4000 0    50   ~ 0
+DATA10
+Text Label 8375 4200 0    50   ~ 0
+DATA11
+Text Label 8375 4300 0    50   ~ 0
+B11
+Text Label 8375 4400 0    50   ~ 0
+G11
+Text Label 8375 4500 0    50   ~ 0
+R11
+Text Label 8375 4600 0    50   ~ 0
+DATA12
+Text Label 8375 4700 0    50   ~ 0
+B12
+Text Label 8375 4800 0    50   ~ 0
+G12
+Text Label 8375 4900 0    50   ~ 0
+R12
+Wire Notes Line
+	950  5825 2025 5825
+Wire Notes Line
+	2025 5825 2025 6350
+Wire Notes Line
+	2025 6350 950  6350
+Wire Notes Line
+	950  6350 950  5825
+Wire Bus Line
+	1250 2225 1250 5650
+Wire Bus Line
+	6225 3400 6225 5650
+Wire Bus Line
+	3725 2475 3725 5650
+Wire Bus Line
+	3275 5650 3275 7325
+Wire Bus Line
+	1250 5650 3275 5650
+Wire Bus Line
+	9150 4975 9150 5600
+Wire Bus Line
+	12525 4500 12525 6900
+Wire Bus Line
+	7550 6900 10325 6900
+Wire Bus Line
+	3325 7625 3325 9150
+Wire Bus Line
+	8750 3175 12550 3175
+Wire Bus Line
+	8750 3175 8750 4800
+Wire Bus Line
+	6175 2225 9825 2225
+Wire Bus Line
+	6175 2225 6175 3875
+Wire Bus Line
+	3675 1250 3675 3625
+Wire Bus Line
+	3675 1250 7450 1250
+Text Notes 950  6450 0    50   ~ 0
+LCD-Display
 $EndSCHEMATC

Commit message: SCL und SCK und Arduino fehlt
Parts:
- J15: footprint Connector_PinHeader_2.54mm:PinHeader_1x01_P2.54mm_Horizontal -> Connector_PinHeader_2.54mm:PinHeader_1x01_P2.54mm_Vertical
- J7: footprint Connector_PinHeader_2.54mm:PinHeader_1x09_P2.54mm_Horizontal -> Connector_PinHeader_2.54mm:PinHeader_1x09_P2.54mm_Vertical
Changed lines of the file:
@@
 F 0 "J15" H 9522 6957 50  0000 R CNN
 F 1 "Conn_01x01_Male" H 9522 7048 50  0000 R CNN
-F 2 "Connector_PinHeader_2.54mm:PinHeader_1x01_P2.54mm_Horizontal" H 9550 7025 50  0001 C CNN
+F 2 "Connector_PinHeader_2.54mm:PinHeader_1x01_P2.54mm_Vertical" H 9550 7025 50  0001 C CNN
 F 3 "~" H 9550 7025 50  0001 C CNN
 	1    9550 7025
@@
 F 0 "J7" H 2658 8206 50  0000 C CNN
 F 1 "Conn_01x09_Male" H 2658 8115 50  0000 C CNN
-F 2 "Connector_PinHeader_2.54mm:PinHeader_1x09_P2.54mm_Horizontal" H 2550 7625 50  0001 C CNN
+F 2 "Connector_PinHeader_2.54mm:PinHeader_1x09_P2.54mm_Vertical" H 2550 7625 50  0001 C CNN
 F 3 "~" H 2550 7625 50  0001 C CNN
 	1    2550 7625
@@
 Wire Notes Line
 	950  6350 950  5825
-Wire Bus Line
-	1250 2225 1250 5650
-Wire Bus Line
-	6225 3400 6225 5650
-Wire Bus Line
-	3725 2475 3725 5650
-Wire Bus Line
-	3275 5650 3275 7325
-Wire Bus Line
-	1250 5650 3275 5650
-Wire Bus Line
-	9150 4975 9150 5600
-Wire Bus Line
-	12525 4500 12525 6900
-Wire Bus Line
-	7550 6900 10325 6900
-Wire Bus Line
-	3325 7625 3325 9150
-Wire Bus Line
-	8750 3175 12550 3175
-Wire Bus Line
-	8750 3175 8750 4800
-Wire Bus Line
-	6175 2225 9825 2225
-Wire Bus Line
-	6175 2225 6175 3875
-Wire Bus Line
-	3675 1250 3675 3625
-Wire Bus Line
-	3675 1250 7450 1250
 Text Notes 950  6450 0    50   ~ 0
 LCD-Display
+Wire Bus Line
+	1250 2225 1250 5650
+Wire Bus Line
+	6225 3400 6225 5650
+Wire Bus Line
+	3725 2475 3725 5650
+Wire Bus Line
+	3275 5650 3275 7325
+Wire Bus Line
+	1250 5650 3275 5650
+Wire Bus Line
+	9150 4975 9150 5600
+Wire Bus Line
+	12525 4500 12525 6900
+Wire Bus Line
+	7550 6900 10325 6900
+Wire Bus Line
+	3325 7625 3325 9150
+Wire Bus Line
+	8750 3175 12550 3175
+Wire Bus Line
+	8750 3175 8750 4800
+Wire Bus Line
+	6175 2225 9825 2225
+Wire Bus Line
+	6175 2225 6175 3875
+Wire Bus Line
+	3675 1250 3675 3625
+Wire Bus Line
+	3675 1250 7450 1250
 $EndSCHEMATC

Commit message: Verbesserung fehlt
Parts:
- C2, C4: footprint Capacitor_SMD:C_1206_3216Metric_Pad1.42x1.75mm_HandSolder -> Capacitor_SMD:C_0805_2012Metric_Pad1.15x1.40mm_HandSolder
- D1: footprint Diode_THT:D_5W_P12.70mm_Horizontal -> Diode_THT:D_5W_P10.16mm_Horizontal
- R5, R7: footprint Resistor_SMD:R_1206_3216Metric_Pad1.42x1.75mm_HandSolder -> Resistor_SMD:R_0805_2012Metric_Pad1.15x1.40mm_HandSolder
Changed lines of the file:
@@
 EESchema Schematic File Version 4
+LIBS:MainPL-cache
 EELAYER 30 0
 EELAYER END
@@
 F 0 "C2" H 6115 8496 50  0000 L CNN
 F 1 "100n" H 6115 8405 50  0000 L CNN
-F 2 "Capacitor_SMD:C_1206_3216Metric_Pad1.42x1.75mm_HandSolder" H 6038 8300 50  0001 C CNN
+F 2 "Capacitor_SMD:C_0805_2012Metric_Pad1.15x1.40mm_HandSolder" H 6038 8300 50  0001 C CNN
 F 3 "~" H 6000 8450 50  0001 C CNN
 	1    6000 8450
@@
 F 0 "R5" H 6275 6800 50  0000 L CNN
 F 1 "1M" H 6400 6775 50  0000 L CNN
-F 2 "Resistor_SMD:R_1206_3216Metric_Pad1.42x1.75mm_HandSolder" V 6355 6775 50  0001 C CNN
+F 2 "Resistor_SMD:R_0805_2012Metric_Pad1.15x1.40mm_HandSolder" V 6355 6775 50  0001 C CNN
 F 3 "~" H 6425 6775 50  0001 C CNN
 	1    6425 6775
@@
 F 0 "C4" H 7440 8721 50  0000 L CNN
 F 1 "100n" H 7440 8630 50  0000 L CNN
-F 2 "Capacitor_SMD:C_1206_3216Metric_Pad1.42x1.75mm_HandSolder" H 7363 8525 50  0001 C CNN
+F 2 "Capacitor_SMD:C_0805_2012Metric_Pad1.15x1.40mm_HandSolder" H 7363 8525 50  0001 C CNN
 F 3 "~" H 7325 8675 50  0001 C CNN
 	1    7325 8675
@@
 F 0 "D1" V 7596 6146 50  0000 R CNN
 F 1 "D" V 7505 6146 50  0000 R CNN
-F 2 "Diode_THT:D_5W_P12.70mm_Horizontal" H 7550 6225 50  0001 C CNN
+F 2 "Diode_THT:D_5W_P10.16mm_Horizontal" H 7550 6225 50  0001 C CNN
 F 3 "~" H 7550 6225 50  0001 C CNN
 	1    7550 6225
@@
 F 0 "R7" V 7343 6000 50  0000 C CNN
 F 1 "10k" V 7434 6000 50  0000 C CNN
-F 2 "Resistor_SMD:R_1206_3216Metric_Pad1.42x1.75mm_HandSolder" V 7480 6000 50  0001 C CNN
+F 2 "Resistor_SMD:R_0805_2012Metric_Pad1.15x1.40mm_HandSolder" V 7480 6000 50  0001 C CNN
 F 3 "~" H 7550 6000 50  0001 C CNN
 	1    7550 6000

Commit message: File gefixed
Connections:
- net INTArduino: no longer U1.6
- net INTB_2: now also U1.4, U1.5; no longer U1.1
- net INTB_3: no longer U1.4
- net at U1.3: no longer U1.5
- net at U3.20 (INTA): now also U1.1
Other:
- moved on the sheet: U1A, U1B
Changed lines of the file:
@@
 EESchema Schematic File Version 4
-LIBS:MainPL-cache
 EELAYER 30 0
 EELAYER END
@@
 Wire Wire Line
 	8725 6150 8725 6250
-Wire Wire Line
-	1400 2725 1475 2725
-Wire Wire Line
-	3850 2975 4150 2975
-Wire Wire Line
-	6400 3900 6575 3900
 $Comp
 L 74xx:74LS32 U1
 U 1 1 5E03B617
-P 4050 4900
-F 0 "U1" V 4004 5088 50  0000 L CNN
-F 1 "74LS32" V 4095 5088 50  0000 L CNN
-F 2 "Package_DIP:DIP-14_W7.62mm_Socket_LongPads" H 4050 4900 50  0001 C CNN
-F 3 "http://www.ti.com/lit/gpn/sn74LS32" H 4050 4900 50  0001 C CNN
-	1    4050 4900
+P 1525 3275
+F 0 "U1" V 1479 3463 50  0000 L CNN
+F 1 "74LS32" V 1570 3463 50  0000 L CNN
+F 2 "Package_DIP:DIP-14_W7.62mm_Socket_LongPads" H 1525 3275 50  0001 C CNN
+F 3 "http://www.ti.com/lit/gpn/sn74LS32" H 1525 3275 50  0001 C CNN
+	1    1525 3275
 	0    1    1    0
 $EndComp
-Wire Wire Line
-	1475 2725 1475 4475
-Wire Wire Line
-	1475 4475 3950 4475
-Wire Wire Line
-	3950 4475 3950 4600
-Connection ~ 1475 2725
-Wire Wire Line
-	1475 2725 1900 2725
-Wire Wire Line
-	4150 4600 4150 2975
-Connection ~ 4150 2975
-Wire Wire Line
-	4150 2975 4425 2975
-Connection ~ 6575 3900
-Wire Wire Line
-	6575 3900 6900 3900
-Wire Wire Line
-	4050 5200 4050 6000
-Wire Wire Line
-	4050 6000 4900 6000
-Wire Wire Line
-	5100 6000 6575 6000
-Wire Wire Line
-	6575 3900 6575 6000
 Wire Bus Line
 	1300 2825 1300 5600
@@
 L 74xx:74LS32 U1
 U 2 1 5E02EBD5
-P 5000 6300
-F 0 "U1" V 4954 6488 50  0000 L CNN
-F 1 "74LS32" V 5045 6488 50  0000 L CNN
-F 2 "Package_DIP:DIP-14_W7.62mm_Socket_LongPads" H 5000 6300 50  0001 C CNN
-F 3 "http://www.ti.com/lit/gpn/sn74LS32" H 5000 6300 50  0001 C CNN
-	2    5000 6300
+P 3975 3400
+F 0 "U1" V 3929 3588 50  0000 L CNN
+F 1 "74LS32" V 4020 3588 50  0000 L CNN
+F 2 "Package_DIP:DIP-14_W7.62mm_Socket_LongPads" H 3975 3400 50  0001 C CNN
+F 3 "http://www.ti.com/lit/gpn/sn74LS32" H 3975 3400 50  0001 C CNN
+	2    3975 3400
 	0    1    1    0
 $EndComp
@@
 Text Notes 950  6450 0    50   ~ 0
 LCD-Display
+Wire Wire Line
+	1400 2725 1425 2725
+Wire Wire Line
+	1425 2975 1425 2725
+Connection ~ 1425 2725
+Wire Wire Line
+	1425 2725 1900 2725
+Wire Wire Line
+	1625 2975 1625 2825
+Wire Wire Line
+	1625 2825 1900 2825
+Wire Wire Line
+	3850 2975 3875 2975
+Wire Wire Line
+	3875 3100 3875 2975
+Connection ~ 3875 2975
+Wire Wire Line
+	3875 2975 4075 2975
+Wire Wire Line
+	4075 3100 4075 2975
 Wire Bus Line
 	1250 2225 1250 5650
@@
 Wire Bus Line
 	3675 1250 7450 1250
+Connection ~ 4075 2975
+Wire Wire Line
+	4075 2975 4425 2975
+Wire Wire Line
+	6400 3900 6900 3900
 $EndSCHEMATC
