File: MainPL/MainPL.sch (KiCad schematic (older format))
At the start: 37 parts, among them J1 Conn_01x06_Female, J10 Conn_01x06_Female, J11 Conn_01x06_Female, J12 Conn_01x06_Female, J13 Conn_01x06_Female, J14 Conn_01x06_Female, J15 Conn_01x01_Male, J16 Conn_01x04_Male, J2 USB_B, J3 Conn_01x06_Female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

Commit message: Add files via upload
V.2 von Parkplatz mit neuen Maßen
Parts:
- removed SW1: SW_Push_Dual, Button_Switch_THT:SW_TH_Tactile_Omron_B3F-10xx, symbol Switch:SW_Push_Dual
- added SW1, SW2: SW_Push_MS, Button_Switch_THT:SW_TH_Tactile_Omron_B3F-10xx, symbol SW_Push_MS:SW_Push_MS
- U1: footprint (none) -> Package_DIP:DIP-14_W7.62mm_Socket_LongPads
Connections:
- net GND: now also SW1.3, SW1.4, SW2.3, SW2.4
- net at D1.2 (A), R7.1, U2.1 (~RESET~/PC6): now also SW2.1, SW2.2
- net at U2.14 (PB0): now also SW1.1, SW1.2
Changed lines of the file:
@@
 EESchema Schematic File Version 4
+LIBS:MainPL-cache
 EELAYER 30 0
 EELAYER END
@@
 Wire Wire Line
 	9525 5075 9250 5075
-$Comp
-L Switch:SW_Push_Dual SW1
-U 1 1 5DFB15DE
-P 8450 6050
-F 0 "SW1" H 8450 6335 50  0000 C CNN
-F 1 "SW_Push_Dual" H 8450 6244 50  0000 C CNN
-F 2 "Button_Switch_THT:SW_TH_Tactile_Omron_B3F-10xx" H 8450 6250 50  0001 C CNN
-F 3 "~" H 8450 6250 50  0001 C CNN
-	1    8450 6050
-	1    0    0    -1
-$EndComp
 Wire Wire Line
 	7775 6125 7950 6125
@@
 Wire Wire Line
 	12075 6650 12075 7600
-Wire Wire Line
-	12075 7600 8800 7600
 Connection ~ 8800 7600
 Wire Wire Line
@@
 F 0 "U1" V 6479 4538 50  0000 L CNN
 F 1 "74LS32" V 6570 4538 50  0000 L CNN
-F 2 "" H 6525 4350 50  0001 C CNN
+F 2 "Package_DIP:DIP-14_W7.62mm_Socket_LongPads" H 6525 4350 50  0001 C CNN
 F 3 "http://www.ti.com/lit/gpn/sn74LS32" H 6525 4350 50  0001 C CNN
 	3    6525 4350
@@
 F 0 "U1" H 1780 8921 50  0000 L CNN
 F 1 "74LS32" H 1780 8830 50  0000 L CNN
-F 2 "" H 1550 8875 50  0001 C CNN
+F 2 "Package_DIP:DIP-14_W7.62mm_Socket_LongPads" H 1550 8875 50  0001 C CNN
 F 3 "http://www.ti.com/lit/gpn/sn74LS32" H 1550 8875 50  0001 C CNN
 	5    1550 8875
@@
 Wire Wire Line
 	5000 4825 6525 4825
-Wire Wire Line
-	6525 4650 6525 4675
+Connection ~ 5000 4825
+Wire Wire Line
+	8800 7600 12075 7600
+Wire Wire Line
+	5550 6950 5525 6950
+Wire Wire Line
+	5525 6950 5525 6750
+Wire Wire Line
+	5525 6750 5550 6750
+Wire Wire Line
+	5525 6950 5525 7175
+Wire Wire Line
+	5525 7175 5750 7175
+Connection ~ 5525 6950
+Wire Wire Line
+	5950 6750 5950 6850
+$Comp
+L power:GND #PWR0107
+U 1 1 5E2D86BA
+P 5950 6850
+F 0 "#PWR0107" H 5950 6600 50  0001 C CNN
+F 1 "GND" H 5955 6677 50  0000 C CNN
+F 2 "" H 5950 6850 50  0001 C CNN
+F 3 "" H 5950 6850 50  0001 C CNN
+	1    5950 6850
+	0    -1   -1   0
+$EndComp
+Connection ~ 5950 6850
+Wire Wire Line
+	5950 6850 5950 6950
+Wire Wire Line
+	6525 4650 6525 4825
 Wire Wire Line
 	3975 3700 3975 4825
@@
 Wire Bus Line
 	3675 1250 7450 1250
-Connection ~ 5000 4825
-Connection ~ 6525 4675
-Wire Wire Line
-	6525 4675 6525 4825
+$Comp
+L SW_Push_MS:SW_Push_MS SW2
+U 1 1 5E336CA3
+P 8450 6050
+F 0 "SW2" H 8450 6335 50  0000 C CNN
+F 1 "SW_Push_MS" H 8450 6244 50  0000 C CNN
+F 2 "Button_Switch_THT:SW_TH_Tactile_Omron_B3F-10xx" H 8450 6250 50  0001 C CNN
+F 3 "~" H 8450 6250 50  0001 C CNN
+	1    8450 6050
+	1    0    0    -1
+$EndComp
+$Comp
+L SW_Push_MS:SW_Push_MS SW1
+U 1 1 5E34020D
+P 5750 6750
+F 0 "SW1" H 5750 7035 50  0000 C CNN
+F 1 "SW_Push_MS" H 5750 6944 50  0000 C CNN
+F 2 "Button_Switch_THT:SW_TH_Tactile_Omron_B3F-10xx" H 5750 6950 50  0001 C CNN
+F 3 "~" H 5750 6950 50  0001 C CNN
+	1    5750 6750
+	1    0    0    -1
+$EndComp
 $EndSCHEMATC
